Commit message: Update ra605 for OpenRAVE IKfast generator

File: sandbox/ra605.urdf (robot description, URDF)
Before this commit: robot ra605_robot, 7 links, 6 joints
Links:
- link base_link: geometry visual cylinder length=0.2 radius=0.105
- link link2: geometry visual cylinder length=0.2 radius=0.090
- link link3: geometry visual cylinder length=0.25 radius=0.08
