Commit message: Update RA605.URDF

File: ra605_description/urdf/ra605.urdf (robot description, URDF)
Before this commit: robot ra605, 7 links, 6 joints
Links:
- link base_link: geometry visual cylinder length=0.375 radius=0.105
- link link2: geometry visual cylinder length=0.34 radius=0.090
- link link3: geometry visual cylinder length=0.338 radius=0.08
Joints:
- joint joint1: limit lower=-3.1416 upper=3.1416 effort=0 velocity=2.618 -> lower=-4.00 upper=1.3 effort=0 velocity=0.555
- joint joint2: limit lower=-3.1416 upper=3.1416 effort=0 velocity=2.618 -> lower=-0.138 upper=3.05 effort=0 velocity=0.555
- joint joint3: limit lower=-3.1416 upper=3.1416 effort=0 velocity=2.618 -> lower=-1.9188 upper=1.9188 effort=0 velocity=0.555
- joint joint4: limit lower=-3.1416 upper=3.1416 effort=0 velocity=2.618 -> lower=-3.1416 upper=3.1416 effort=0 velocity=0.555
- joint joint5: limit lower=-3.1416 upper=3.1416 effort=0 velocity=2.618 -> lower=-1.9188 upper=1.9188 effort=0 velocity=0.555
- joint joint6: limit lower=-3.1416 upper=3.1416 effort=0 velocity=2.618 -> lower=-3.1416 upper=3.1416 effort=0 velocity=0.555

Commit message: Update URDF and related config files for RA605

File: ra605_description/urdf/ra605.urdf (robot description, URDF)
Before this commit: robot ra605, 7 links, 6 joints
Links:
- link link5: geometry visual box size=0.070 0.16 0.086
Joints:
- joint joint1: limit lower=-4.00 upper=1.3 effort=0 velocity=0.555 -> lower=-2.88 upper=2.88 effort=0 velocity=0.555
- joint joint2: limit lower=-0.138 upper=3.05 effort=0 velocity=0.555 -> lower=-2.0071 upper=1.4835 effort=0 velocity=0.555
- joint joint3: limit lower=-1.9188 upper=1.9188 effort=0 velocity=0.555 -> lower=-2.4085 upper=1.8675 effort=0 velocity=0.555; origin xyz=0.34 0 0 rpy=0 0 0 -> xyz=0 0 0.34 rpy=0 0 0
- joint joint4: axis 1 0 0 -> 0 0 1; origin xyz=0.338 0 0.04 rpy=0 0 0 -> xyz=-0.04 0 0.338 rpy=0 0 0
- joint joint5: limit lower=-1.9188 upper=1.9188 effort=0 velocity=0.555 -> lower=-2.0071 upper=2.0071 effort=0 velocity=0.555
- joint joint6: axis 1 0 0 -> 0 0 1; origin xyz=0.086 0 0 rpy=0 0 0 -> xyz=0 0 0.086 rpy=0 0 0
